Commit message: Added imu sensor to test_cart_position urdf

File: gazebo_ros2_control_demos/urdf/test_cart_position.xacro.urdf (robot description, URDF)
Before this commit: robot cartopole, 3 links, 2 joints
Links:
- added link imu, mass 0.1
Joints:
- added joint cart_to_imu: type fixed, parent cart, child imu, origin xyz=0.0 0.0 0.0

Commit message: Remove IMU from position cart, and cleanup velocity cart

File: gazebo_ros2_control_demos/urdf/test_cart_position.xacro.urdf (robot description, URDF)
Before this commit: robot cartopole, 4 links, 3 joints
Links:
- removed link imu
Joints:
- removed joint cart_to_imu
