Commit message: Fix mimic definition from URDF

File: gazebo_ros2_control_demos/urdf/test_gripper_mimic_joint_effort.xacro.urdf (robot description, URDF)
Before this commit: robot gripper, 4 links, 3 joints
Joints:
- joint left_finger_joint: mimic joint=right_finger_joint -> joint=right_finger_joint multiplier=1 offset=0

File: gazebo_ros2_control_demos/urdf/test_gripper_mimic_joint_position.xacro.urdf (robot description, URDF)
Before this commit: robot gripper, 4 links, 3 joints
Joints:
- joint left_finger_joint: mimic joint=right_finger_joint -> joint=right_finger_joint multiplier=1 offset=0
