Commit message: Fix inertias by introducing a macro

File: gazebo_ros2_control_demos/urdf/test_pendulum_effort.xacro.urdf (robot description, URDF)
Before this commit: robot cartopole, 4 links, 3 joints
Links:
- removed link cart
- removed link pendulum
Joints:
- joint cart_to_pendulum: limit lower=-10000 upper=10000 effort=1000.0 velocity=30 -> lower=-100000 upper=100000 effort=10000.0 velocity=100000; origin xyz=0.0 0.35 0.0 -> xyz=0.0 0.35 0.0 rpy=0 0 0

Commit message: Fix origin in macro and set some damping

File: gazebo_ros2_control_demos/urdf/test_pendulum_effort.xacro.urdf (robot description, URDF)
Before this commit: robot pendulum on cart, 2 links, 3 joints
Joints:
- joint cart_to_pendulum: origin xyz=0.0 0.35 0.0 rpy=0 0 0 -> xyz=0.0 0.35 0.0 rpy=0 0.1 0

Commit message: Change initial pose of pendulum

File: gazebo_ros2_control_demos/urdf/test_pendulum_effort.xacro.urdf (robot description, URDF)
Before this commit: robot pendulum on cart, 2 links, 3 joints
Joints:
- joint cart_to_pendulum: origin xyz=0.0 0.35 0.0 rpy=0 0.1 0 -> xyz=0.0 0.35 0.0 rpy=0 ${pi} 0

File: gazebo_ros2_control_demos/urdf/test_pendulum_position.xacro.urdf (robot description, URDF)
Before this commit: robot pendulum on cart, 2 links, 3 joints
Joints:
- joint cart_to_pendulum: origin xyz=0.0 0.35 0.0 rpy=0 0.1 0 -> xyz=0.0 0.35 0.0 rpy=0 ${pi} 0
